Commit message: model update

File: src/triton_gazebo/models/triton_auv/model.urdf (robot description, URDF)
Before this commit: robot steelhead_urdf, 7 links, 6 joints
Links:
- added link imu_link
Joints:
- added joint imu_joint: type fixed, parent base_link, child imu_link, origin xyz=0 0.25 0 rpy=0 0 0
