Commit message: depth camera simulation

File: src/steelhead_controls/models/steelhead_auv/model.urdf (robot description, URDF)
Before this commit: robot steelhead_urdf, 8 links, 7 joints
Links:
- added link camera_link; visual box size=0.05 0.05 0.05
- added link camera_link_optical
Joints:
- added joint camera_joint: type fixed, parent base_link, child camera_link, origin xyz=0.45 -0.06 0 rpy=0 0 0
- added joint camera_optical_joint: type fixed, parent camera_link, child camera_link_optical, origin xyz=0 0 0 rpy=-1.5708 0 -1.5708

Commit message: Rename files

File: src/steelhead_controls/models/steelhead_auv/model.urdf (robot description, URDF)
Before this commit: robot steelhead_urdf, 10 links, 9 joints
Links:
- link base_link: geometry collision mesh filename=package://spiderfish_urdf/meshes/base_link.STL; visual mesh filename=package://spiderfish_urdf/meshes/base_link.STL
- link thruster-1_link: geometry collision mesh filename=package://spiderfish_urdf/meshes/thruster-1_link.STL; visual mesh filename=package://spiderfish_urdf/meshes/thruster-1_link.STL
- link thruster-2_link: geometry collision mesh filename=package://spiderfish_urdf/meshes/thruster-2_link.STL; visual mesh filename=package://spiderfish_urdf/meshes/thruster-2_link.STL
- link thruster-3_link: geometry collision mesh filename=package://spiderfish_urdf/meshes/thruster-3_link.STL; visual mesh filename=package://spiderfish_urdf/meshes/thruster-3_link.STL
- link thruster-6_link: geometry collision mesh filename=package://spiderfish_urdf/meshes/thruster-6_link.STL; visual mesh filename=package://spiderfish_urdf/meshes/thruster-6_link.STL
- link thruster_4_link: geometry collision mesh filename=package://spiderfish_urdf/meshes/thruster_4_link.STL; visual mesh filename=package://spiderfish_urdf/meshes/thruster_4_link.STL
- link thruster_5_link: geometry collision mesh filename=package://spiderfish_urdf/meshes/thruster_5_link.STL; visual mesh filename=package://spiderfish_urdf/meshes/thruster_5_link.STL
